Commit message: Adjust basic amcl and navigation parameters
Adjustments based on the lesson explanation.
With current paramenters, if the robot does not get stuck inside the inflation area, it can sometimes reach the goal.

File: urdf/udacity_bot.xacro (robot description, xacro)
@@ -70,5 +70,5 @@
     </collision>
     <visual name='left_wheel_visual'>
-      <origin xyz="0 0 0" rpy="1.5705 0 0"/>
+      <origin xyz="0 0 0" rpy="1.5707 0 0"/>
       <geometry>
         <cylinder radius="0.1" length="0.05"/>
