Commit message: Fix instability by extending the casters
Adjust colision space of robot's head

File: urdf/r2d2_bot.xacro (robot description, xacro)
@@ -44,5 +44,5 @@
       <origin xyz="0 0.11 -0.07" rpy=" 0 0 0"/>
       <geometry>
-        <box size="0.2 0.02 0.04"/>
+        <box size="0.4 0.02 0.04"/>
       </geometry>
     </collision>
@@ -50,5 +50,5 @@
       <origin xyz="0 0.11 -0.07" rpy=" 0 0 0"/>
       <geometry>
-        <box size="0.2 0.02 0.04"/>
+        <box size="0.4 0.02 0.04"/>
       </geometry>
       <material name="blue"/>
@@ -57,5 +57,5 @@
       <origin xyz="0 -0.11 -0.07" rpy=" 0 0 0"/>
       <geometry>
-        <box size="0.2 0.02 0.04"/>
+        <box size="0.4 0.02 0.04"/>
       </geometry>
     </collision>
@@ -63,10 +63,10 @@
       <origin xyz="0 -0.11 -0.07" rpy=" 0 0 0"/>
       <geometry>
-        <box size="0.2 0.02 0.04"/>
+        <box size="0.4 0.02 0.04"/>
       </geometry>
       <material name="blue"/>
     </visual>
     <collision name='fl_caster_collision'>
-      <origin xyz="0.095 0.11 -0.09" rpy=" 0 0 0"/>
+      <origin xyz="0.195 0.11 -0.09" rpy=" 0 0 0"/>
       <geometry>
         <sphere radius="0.0099"/>
@@ -74,5 +74,5 @@
     </collision>
     <visual name='fl_caster_visual'>
-      <origin xyz="0.095 0.11 -0.09" rpy=" 0 0 0"/>
+      <origin xyz="0.195 0.11 -0.09" rpy=" 0 0 0"/>
       <geometry>
         <sphere radius="0.0099"/>
@@ -80,5 +80,5 @@
     </visual>
     <collision name='bl_caster_collision'>
-      <origin xyz="-0.095 0.11 -0.09" rpy=" 0 0 0"/>
+      <origin xyz="-0.195 0.11 -0.09" rpy=" 0 0 0"/>
       <geometry>
         <sphere radius="0.0099"/>
@@ -86,5 +86,5 @@
     </collision>
     <visual name='bl_caster_visual'>
-      <origin xyz="-0.095 0.11 -0.09" rpy=" 0 0 0"/>
+      <origin xyz="-0.195 0.11 -0.09" rpy=" 0 0 0"/>
       <geometry>
         <sphere radius="0.0099"/>
@@ -92,5 +92,5 @@
     </visual>
     <collision name='fr_caster_collision'>
-      <origin xyz="0.095 -0.11 -0.09" rpy=" 0 0 0"/>
+      <origin xyz="0.195 -0.11 -0.09" rpy=" 0 0 0"/>
       <geometry>
         <sphere radius="0.0099"/>
@@ -98,5 +98,5 @@
     </collision>
     <visual name='fr_caster_visual'>
-      <origin xyz="0.095 -0.11 -0.09" rpy=" 0 0 0"/>
+      <origin xyz="0.195 -0.11 -0.09" rpy=" 0 0 0"/>
       <geometry>
         <sphere radius="0.0099"/>
@@ -104,5 +104,5 @@
     </visual>
     <collision name='br_caster_collision'>
-      <origin xyz="-0.095 -0.11 -0.09" rpy=" 0 0 0"/>
+      <origin xyz="-0.195 -0.11 -0.09" rpy=" 0 0 0"/>
       <geometry>
         <sphere radius="0.0099"/>
@@ -110,37 +110,13 @@
     </collision>
     <visual name='br_caster_visual'>
-      <origin xyz="-0.095 -0.11 -0.09" rpy=" 0 0 0"/>
-      <geometry>
-        <sphere radius="0.0099"/>
-      </geometry>
-    </visual>
-    <!--collision name='back_caster_collision'>
-      <origin xyz="-0.05 0 -0.05" rpy=" 0 0 0"/>
-      <geometry>
-        <sphere radius="0.0499"/>
-      </geometry>
-    </collision>
-    <visual name='back_caster_visual'>
-      <origin xyz="-0.05 0 -0.05" rpy=" 0 0 0"/>
-      <geometry>
-        <sphere radius="0.05"/>
-      </geometry>
-    </visual>
-    <collision name='front_caster_collision'>
-      <origin xyz="0.05 0 -0.05" rpy=" 0 0 0"/>
-      <geometry>
-        <sphere radius="0.0499"/>
-      </geometry>
-    </collision>
-    <visual name='front_caster_visual'>
-      <origin xyz="0.05 0 -0.05" rpy=" 0 0 0"/>
-      <geometry>
-        <sphere radius="0.05"/>
-      </geometry>
-    </visual-->
+      <origin xyz="-0.195 -0.11 -0.09" rpy=" 0 0 0"/>
+      <geometry>
+        <sphere radius="0.0099"/>
+      </geometry>
+    </visual>
     <collision name='head_colision'>
-      <origin xyz="0 0 0.35" rpy=" 0 0 0"/>
-      <geometry>
-        <sphere radius="0.0499"/>
+      <origin xyz="0 0 0.25" rpy=" 0 0 0"/>
+      <geometry>
+        <sphere radius="0.1"/>
       </geometry>
     </collision>
